File: adv-w20.sch (EAGLE design)
At the start: 4 parts

Commit message: Add files via upload
Parts:
- added C1: 1uF, may2019-teaching:C_CHIP
- added C10, C2, C7, C8, C9: 0.1uF, may2019-teaching:C_CHIP
- added C5, C6: 22pF, may2019-teaching:C_CHIP
- added Q1, Q2: NPN, may2019-teaching:NPN
- added R3, R4, R7: 10k, may2019-teaching:R_CHIP
- added R5, R6: R_CHIP, may2019-teaching:R_CHIP
- added S3, S4: (no value), may2019-teaching:TAC_SWITCHPTH
- added U1: ESP32-WROOM, adv-w20:ESP32-WROOM
- added U3: CH340G, may2019-teaching:CH340G
- added Y1: 12MHz, adafruit:CRYSTALHC49S
- renumbered U$2 to U2
Connections:
- new net BOOT: C8.1, Q2.C, R6.1, S4.3, S4.4, U1.IO0
- new net DTR: Q2.E, R3.1, U3.DTR#
- new net EN: C7.1, Q1.C, R5.1, S3.3, S3.4
- new net MCU-RX: U1.RXD0, U3.TXD
- new net MCU-TX: U1.TXD0, U3.RXD
- new net N$2: C6.1, U3.XI, Y1.2
- new net N$3: C1.1, C2.1, U3.V3, U3.VCC
- new net N$4: Q2.B, R4.1
- new net N$5: C9.1, R7.1, U1.3V3
- new net N$6: C10.1, R7.2, U1.EN
- new net N$7: Q1.B, R3.2
- new net N$8: C7.2, S3.1, S3.2
- new net N$9: C8.2, S4.1, S4.2
- new net RTS: Q1.E, R4.2, U3.RTS#
- new net USB-D+: U3.UD+
- new net USB-D-: U3.UD-
- new net XO: C5.1, U3.XO, Y1.1
Other:
- note added: "1.0"
- note added: "Andy Monk"
- note added: "GPS Clock"

Commit message: Add files via upload
Connections:
- removed net N$3: C1.1, C2.1, U3.V3, U3.VCC
- removed net N$5: C9.1, R7.1, U1.3V3
- removed net N$8: C7.2, S3.1, S3.2
- removed net N$9: C8.2, S4.1, S4.2
- net GND: now also C1.2, C10.2, C2.2, C5.2, C6.2, C7.2, C8.2, C9.2, S3.1, S3.2, S4.1, S4.2, U1.GND, U3.GND
- net VCC: now also C1.1, C2.1, C9.1, R5.2, R6.2, R7.1, U1.3V3, U3.V3, U3.VCC

Commit message: Add files via upload
Parts:
- added C11: 0.1uF, may2019-teaching:C_CHIP
- added C3, C4: 9pF, may2019-teaching:C_CHIP
- added R10, R8, R9: 4.7k, may2019-teaching:R_CHIP
- added U$19: MCP7940M-MSOP8, adv-w20:MCP7940M-MSOP8
- added U$26: USB-MICRO-B, may2019-teaching:USB-MICRO-B
- added Y2: 32.768kHz, adv-w20:XTAL
- R5, R6: value R_CHIP -> 10k
Connections:
- removed net N$6: C10.1, R7.2, U1.EN
- removed net RST: R2.2, U2.RST
- new net GPS_RST: R2.2, U1.IO19, U2.RST
- new net MFP: R10.1, U$19.MFP, U1.IO23
- new net N$3: C4.1, U$19.X1, Y2.2
- new net SCL: R8.1, U$19.SCL, U1.IO22
- new net SDA: R9.1, U$19.SDA, U1.IO21
- new net X2: C3.1, U$19.X2, Y2.1
- net EN: now also C10.1, R7.2, U1.EN
- net GND: now also C11.2, C3.2, C4.2, U$19.GND
- net GPS_PPS: now also U1.IO18
- net GPS_RX: now also U1.IO16
- net GPS_TX: now also U1.IO17
- net VCC: now also C11.1, R10.2, R8.2, R9.2, U$19.VCC
Other:
- moved on the sheet: C1, C10, C2, C5, C6, C7, C8, C9, Q1, Q2, R1, R2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
